File: LEDIndicators.kicad_sch (KiCad schematic)
At the start: 2 parts

Commit message: 2nd rev schematic done
Parts:
- R10: value 4.7k -> 1k; Distributor Prt # 311-4.7KJRCT-ND -> 311-1.0KJRCT-ND; Manuf Prt # RC0402JR-074K7L -> RC0402JR-071KL
Changed lines of the file:
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@@
 			)
 		)
-		(property "Value" "4.7k"
+		(property "Value" "1k"
 			(at 139.192 82.804 90)
 			(effects
@@
 			)
 		)
-		(property "Description" "RES 4.7K OHM 5% 1/16W 0402"
+		(property "Description" "RES 1K OHM 5% 1/16W 0402"
 			(at 137.16 82.55 0)
 			(effects
@@
 			)
 		)
-		(property "Distributor Prt #" "311-4.7KJRCT-ND"
+		(property "Distributor Prt #" "311-1.0KJRCT-ND"
 			(at 137.16 82.55 0)
 			(effects
@@
 			)
 		)
-		(property "Manuf Prt #" "	 RC0402JR-074K7L"
+		(property "Manuf Prt #" "RC0402JR-071KL"
 			(at 137.16 82.55 0)
 			(effects
