File: Irrigation.kicad_sch (KiCad schematic)
At the start: 8 parts, among them J6 OSTVN02A150, J7 Conn_01x03, U11 DRV8838DSGR, U8 TPS22914BYFPR

Commit message: updated schematic for pwr savings
Parts:
- added R22: 4.7k, Resistor_SMD:R_0402_1005Metric, symbol Device:R_Small_US
Connections:
- net FLOW_SNS_ENA: now also R22.2
- net GND: now also R22.1
Other:
- title: SproutSyncProto-A-01 -> SproutSyncProto-A-02

Commit message: updated pcb for pwr savings
Other:
- title: SproutSyncProto-A-02 -> SproutSyncProto-A-04
Changed lines of the file:
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@@
 	(paper "A4")
 	(title_block
-		(title "SproutSyncProto-A-02")
-		(date "2026-04-29")
+		(title "SproutSyncProto-A-04")
+		(date "2026-05-04")
 		(rev "0.2")
 		(company "SproutSync LTD")
