File: SoilSense.kicad_sch (KiCad schematic)
At the start: 30 parts, among them J3 OSTVN04A150, U10 SN74LVC1T45DBVR, U12 SN74LVC1T45DBVR, U2 TPS22914BYFPR, U4 SN65HVD3082EDR

Commit message: replaced soil_sns frontend with SN74
Parts:
- U10, U12: footprint SN74LVC1T45DBVR:SOT95P280X145-6N -> SproutSenseFootprints:SOT95P280X145-6N; Distributor Prt # (none) -> 296-16843-1-ND; Manuf Prt # (none) -> SN74LVC1T45DBVR
Changed lines of the file:
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@@
 			)
 		)
-		(property "Footprint" "SN74LVC1T45DBVR:SOT95P280X145-6N"
+		(property "Footprint" "SproutSenseFootprints:SOT95P280X145-6N"
 			(at 59.69 66.04 0)
 			(effects
@@
 			)
 		)
-		(property "Datasheet" ""
+		(property "Datasheet" "https://www.ti.com/lit/ds/symlink/sn74lvc1t45.pdf?ts=1765853339100&ref_url=https%253A%252F%252Fwww.ti.com%252Fproduct%252FSN74LVC1T45%253Futm_source%253Dgoogle%2526utm_medium%253Dcpc%2526utm_campaign%253Dasc-int-null-44700045345892941_prodfolderdynamic-cpc-pf-google-tw_zhtw_int%2526utm_content%253Dprodfolddynamic%2526ds_k%253DDYNAMIC+SEARCH+ADS%2526DCM%253Dyes%2526gclsrc%253Daw.ds%2526gad_source%253D1%2526gad_campaignid%253D13696973196%2526gclid%253DCj0KCQiAgP_JBhD-ARIsANpEMxxV_UbqxExnx1mvuNtffIm9WmyZz6MwMfzZUxsiR6oqkjohx3sVblcaAiefEALw_wcB#page=6.09"
 			(at 59.69 66.04 0)
 			(effects
@@
 			)
 		)
-		(property "Description" ""
+		(property "Description" "IC XLTR VL BIDIR SOT-23-6"
+			(at 59.69 66.04 0)
+			(effects
+				(font
+					(size 1.27 1.27)
+				)
+				(hide yes)
+			)
+		)
+		(property "Distributor Prt #" "296-16843-1-ND"
+			(at 59.69 66.04 0)
+			(effects
+				(font
+					(size 1.27 1.27)
+				)
+				(hide yes)
+			)
+		)
+		(property "Manuf Prt #" "SN74LVC1T45DBVR"
 			(at 59.69 66.04 0)
 			(effects
@@
 			)
 		)
-		(property "Footprint" "SN74LVC1T45DBVR:SOT95P280X145-6N"
+		(property "Footprint" "SproutSenseFootprints:SOT95P280X145-6N"
 			(at 60.96 110.49 0)
 			(effects
@@
 			)
 		)
-		(property "Datasheet" ""
+		(property "Datasheet" "https://www.ti.com/lit/ds/symlink/sn74lvc1t45.pdf?ts=1765853339100&ref_url=https%253A%252F%252Fwww.ti.com%252Fproduct%252FSN74LVC1T45%253Futm_source%253Dgoogle%2526utm_medium%253Dcpc%2526utm_campaign%253Dasc-int-null-44700045345892941_prodfolderdynamic-cpc-pf-google-tw_zhtw_int%2526utm_content%253Dprodfolddynamic%2526ds_k%253DDYNAMIC+SEARCH+ADS%2526DCM%253Dyes%2526gclsrc%253Daw.ds%2526gad_source%253D1%2526gad_campaignid%253D13696973196%2526gclid%253DCj0KCQiAgP_JBhD-ARIsANpEMxxV_UbqxExnx1mvuNtffIm9WmyZz6MwMfzZUxsiR6oqkjohx3sVblcaAiefEALw_wcB#page=6.09"
 			(at 60.96 110.49 0)
 			(effects
@@
 			)
 		)
-		(property "Description" ""
+		(property "Description" "IC XLTR VL BIDIR SOT-23-6"
 			(at 60.96 110.49 0)
 			(effects
+				(font
+					(size 1.27 1.27)
+				)
+				(hide yes)
+			)
+		)
+		(property "Distributor Prt #" "296-16843-1-ND"
+			(at 60.96 110.49 0)
+			(effects
+				(font
+					(size 1.27 1.27)
+				)
+				(hide yes)
+			)
+		)
+		(property "Manuf Prt #" "SN74LVC1T45DBVR"
+			(at 60.96 110.49 0)
+			(effects

Commit message: ver2 layout in progress
Parts:
- removed D1, D2, D3: DESD5V0S1BA-7, Diode_SMD:D_SOD-323, symbol Device:D_TVS
- removed R4, R5: 4.7k, Resistor_SMD:R_0402_1005Metric, symbol Device:R_Small_US
- added R26: 9.31k, Resistor_SMD:R_0402_1005Metric, symbol Device:R_Small_US
- added U14: CDSOT23-SM712, SproutSenseFootprints:SOT_SM712, symbol SproutSense:CDSOT23-SM712
Connections:
- net +5V: no longer C8.1, U4.8 (VCC)
- net GND: now also R26.1, U14.3 (common)
- net RS485_A+: now also U14.1 (A1)
- net RS485_B-: now also U14.2 (A2)
- net SOIL_PWR_5p0: now also C8.1, U4.8 (VCC)
- net WRT_ENA: now also R26.2
Other:
- moved on the sheet: R12, R3

Commit message: rev2 precheck DRC clean
Parts:
- TP1, TP12, TP2, TP3, TP4, TP5, TP6: footprint TestPoint:TestPoint_Pad_D1.0mm -> TestPoint:TestPoint_THTPad_1.0x1.0mm_Drill0.5mm
Changed lines of the file:
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@@
 			)
 		)
-		(property "Footprint" "TestPoint:TestPoint_Pad_D1.0mm"
+		(property "Footprint" "TestPoint:TestPoint_THTPad_1.0x1.0mm_Drill0.5mm"
 			(at 45.72 101.6 0)
 			(effects
@@
 			)
 		)
-		(property "Footprint" "TestPoint:TestPoint_Pad_D1.0mm"
+		(property "Footprint" "TestPoint:TestPoint_THTPad_1.0x1.0mm_Drill0.5mm"
 			(at 254 118.11 0)
 			(effects
@@
 			)
 		)
-		(property "Footprint" "TestPoint:TestPoint_Pad_D1.0mm"
+		(property "Footprint" "TestPoint:TestPoint_THTPad_1.0x1.0mm_Drill0.5mm"
 			(at 68.58 139.7 0)
 			(effects
@@
 			)
 		)
-		(property "Footprint" "TestPoint:TestPoint_Pad_D1.0mm"
+		(property "Footprint" "TestPoint:TestPoint_THTPad_1.0x1.0mm_Drill0.5mm"
 			(at 248.92 113.03 0)
 			(effects
@@
 			)
 		)
-		(property "Footprint" "TestPoint:TestPoint_Pad_D1.0mm"
+		(property "Footprint" "TestPoint:TestPoint_THTPad_1.0x1.0mm_Drill0.5mm"
 			(at 63.5 137.16 0)
 			(effects
@@
 			)
 		)
-		(property "Footprint" "TestPoint:TestPoint_Pad_D1.0mm"
+		(property "Footprint" "TestPoint:TestPoint_THTPad_1.0x1.0mm_Drill0.5mm"
 			(at 140.97 53.34 0)
 			(effects
@@
 			)
 		)
-		(property "Footprint" "TestPoint:TestPoint_Pad_D1.0mm"
+		(property "Footprint" "TestPoint:TestPoint_THTPad_1.0x1.0mm_Drill0.5mm"
 			(at 40.64 58.42 0)
 			(effects

Commit message: add diode cathode indicator
Parts:
- J3: now not fitted
Changed lines of the file:
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@@
 		(in_bom yes)
 		(on_board yes)
-		(dnp no)
+		(dnp yes)
 		(fields_autoplaced yes)
 		(property "Reference" "J3"

Commit message: updated schematic for pwr savings
Parts:
- removed J3: OSTVN04A150, SproutSenseFootprints:CONN_OSTVN04A150_OST, symbol Connector:Screw_Terminal_01x04
- removed R2, R6: 1k, Resistor_SMD:R_0402_1005Metric, symbol Device:R_Small_US
- added J1: TBP02R1-381-04BE, TBP02R1-381-04BE:CUI_TBP02R1-381-04BE, symbol SproutSense:TBP02R1-381-04BE
- added R23, R24, R28: 4.7k, Resistor_SMD:R_0402_1005Metric, symbol Device:R_Small_US
Connections:
- net GND: now also J1.4, R23.1
- net RS485_A+: now also J1.3
- net RS485_B-: now also J1.2
- net RX: now also R28.2
- net SOIL_PWR_5p0: now also J1.1
- net SOIL_SNS_ENA: now also R23.2
- net TX: now also R24.2
- net at D4.2 (A): now also R28.1
- net at D5.2 (A): now also R24.1
Other:
- title: SproutSyncProto-A-01 -> SproutSyncProto-A-02

Commit message: updated pcb for pwr savings
Parts:
- removed TP3, TP4: TestPoint, TestPoint:TestPoint_THTPad_1.0x1.0mm_Drill0.5mm, symbol Connector:TestPoint
- J1: footprint TBP02R1-381-04BE:CUI_TBP02R1-381-04BE -> SproutSenseFootprints:CUI_TBP02R1-381-04BE
Other:
- title: SproutSyncProto-A-02 -> SproutSyncProto-A-04
