File: SoilSense.kicad_sch (KiCad schematic)
At the start: 26 parts, among them J1 TBP02R1-381-04BE, U10 SN74LVC1T45DBVR, U12 SN74LVC1T45DBVR, U14 CDSOT23-SM712, U2 TPS22914BYFPR, U4 SN65HVD3082EDR

Commit message: mutli soil sensor update
Parts:
- removed C2, C22, C23, C24: 1uF, Capacitor_SMD:C_0402_1005Metric, symbol Device:C_Small
- removed TP1, TP2: TestPoint, TestPoint:TestPoint_THTPad_1.0x1.0mm_Drill0.5mm, symbol Connector:TestPoint
- removed U10, U12: SN74LVC1T45DBVR, SproutSenseFootprints:SOT95P280X145-6N, symbol SproutSense:SN74LVC1T45DBVR
- added C18, C20, C21, C31, C34, C35: 1uF, Capacitor_SMD:C_0402_1005Metric, symbol Device:C_Small
- added C30, C32, C33: 22uF, Capacitor_SMD:C_0402_1005Metric, symbol Device:C_Small
- added C36, C37: 100nF, Capacitor_SMD:C_0402_1005Metric, symbol Device:C_Small
- added J2, J6, J7: TBP02R1-381-04BE, SproutSenseFootprints:CUI_TBP02R1-381-04BE, symbol SproutSense:TBP02R1-381-04BE
- added R13, R15, R17: 0, Resistor_SMD:R_0402_1005Metric, symbol Device:R_Small_US
- added R16, R36, R6: 120, Resistor_SMD:R_0402_1005Metric, symbol Device:R_Small_US
- added R33, R34, R35: 9.31k, Resistor_SMD:R_0402_1005Metric, symbol Device:R_Small_US
- added R37, R38, R39: 4.7k, Resistor_SMD:R_0402_1005Metric, symbol Device:R_Small_US
- added TP13, TP16, TP17: TestPoint, TestPoint:TestPoint_THTPad_1.0x1.0mm_Drill0.5mm, symbol Connector:TestPoint
- added U11, U18, U19: SN65HVD3082EDR, SproutSenseFootprints:SOIC127P599X175-8N, symbol SproutSense:SN65HVD3082EDR
- added U17, U20, U21: CDSOT23-SM712, SproutSenseFootprints:SOT_SM712, symbol SproutSense:CDSOT23-SM712
- added U22, U23, U24: TPS22914BYFPR, SproutSenseFootprints:YFP4_TEX, symbol SproutSense:TPS22914BYFPR
- added U25: NXU0202DCH, Package_SO:VSSOP-8_2.3x2mm_P0.5mm, symbol SproutSense:NXB0101
Connections:
- net +3V3: now also C36.1, U25.3 (VCC_A)
- net +5V: now also C30.1, C32.1, C33.1, C37.1, U22.A2 (VIN), U23.A2 (VIN), U24.A2 (VIN), U25.7 (VCC_B)
- net GND: now also C18.2, C20.2, C21.2, C30.2, C31.2, C32.2, C33.2, C34.2, C35.2, C36.2, C37.2, J2.4, J6.4, J7.4, R33.1, R34.1, R35.1, R37.1, R38.1, R39.1, U11.5 (GND), U17.3 (common), U18.5 (GND), U19.5 (GND), U20.3 (common), U21.3 (common), U22.B1 (GND), U23.B1 (GND), U24.B1 (GND), U25.2 (GND)
- net RX: now also U11.1 (R), U18.1 (R), U19.1 (R), U25.8 (YB1)
- net SOIL_SNS_ENA: now also R37.2, R38.2, R39.2, U22.B2 (ON), U23.B2 (ON), U24.B2 (ON)
- net TX: now also U11.4 (D), U18.4 (D), U19.4 (D), U25.4 (YA2)
- net UART_RX: now also U25.1 (B2)
- net UART_TX: now also U25.5 (A1)
- net WRT_ENA: now also R33.2, R34.2, R35.2, TP13.1, TP16.1, TP17.1, U11.2 (~{RE}), U11.3 (DE), U18.2 (~{RE}), U18.3 (DE), U19.2 (~{RE}), U19.3 (DE)
- net RS485_A+: no longer names the net of R12.2, U14.1 (A1), U4.6 (A)
- net RS485_A+: now also J1.2; no longer J1.3
- net RS485_B-: no longer names the net of R3.1, U14.2 (A2), U4.7 (B)
- net RS485_B-: now also J1.3; no longer J1.2
- net SOIL_PWR_5p0 renamed +SOIL2V
- new net: J6.2, R15.2, U18.6 (A), U20.1 (A1)
- new net: J6.3, R16.1, U18.7 (B), U20.2 (A2)
- new net: R17.1, R36.2
- new net: J7.2, R17.2, U19.6 (A), U21.1 (A1)
- new net: J2.3, R6.1, U11.7 (B), U17.2 (A2)
- new net: R13.1, R6.2
- new net: J2.2, R13.2, U11.6 (A), U17.1 (A1)
- new net: J7.3, R36.1, U19.7 (B), U21.2 (A2)
- new net: R15.1, R16.2
- new net +SOIL1V: C18.1, C31.1, J2.1, U11.8 (VCC), U22.A1 (VOUT)
- new net +SOIL3V: C20.1, C34.1, J6.1, U18.8 (VCC), U23.A1 (VOUT)
- new net +SOIL4V: C21.1, C35.1, J7.1, U19.8 (VCC), U24.A1 (VOUT)
- new net LVL_SHFT_EN: U25.6 (OE)
Other:
- moved on the sheet: C10, C7, C8, D4, D5, J1, R12, R23, R24, R26, R28, R3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
