File: UserPeriphs.kicad_sch (KiCad schematic)
At the start: 4 parts

Commit message: updated schematic for pwr savings
Other:
- title: SproutSyncProto-A-01 -> SproutSyncProto-A-02

Commit message: updated pcb for pwr savings
Other:
- title: SproutSyncProto-A-02 -> SproutSyncProto-A-04
Changed lines of the file:
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@@
 	(paper "A4")
 	(title_block
-		(title "SproutSyncProto-A-02")
-		(date "2026-04-29")
+		(title "SproutSyncProto-A-04")
+		(date "2026-05-04")
 		(rev "0.2")
 		(company "SproutSync LTD")
