File: SproutSync_SensorNode.kicad_pcb (KiCad board)
At the start: 2 copper layers, 61.7 x 81 mm, 100 parts, among them J1 TBP02R1-381-04BE, J2 BM04B-SRSS-TB, J3 Conn_01x01_Socket, J4 10132797-031100LF, J5 10132797-031100LF, J6 OSTVN02A150, J7 Conn_01x03, J8 Conn_ARM_JTAG_SWD_10, J9 Conn_01x01_Socket, Q1 CSD15380F3T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

Commit message: added vias
Routing:
- net IRRI_PWR_5p0: track 36.1 -> 37.4 mm
- net /PetalStackingConectors/PAD15: track 84.0 -> 85.3 mm
- net GND: vias 23 -> 101
