File: SproutSync_SensorNode.kicad_pcb (KiCad board)
At the start: 2 copper layers, 61.7 x 81 mm, 100 parts, among them J1 TBP02R1-381-04BE, J2 BM04B-SRSS-TB, J3 Conn_01x01_Socket, J4 10132797-031100LF, J5 10132797-031100LF, J6 OSTVN02A150, J7 Conn_01x03, J8 Conn_ARM_JTAG_SWD_10, J9 Conn_01x01_Socket, Q1 CSD15380F3T, Q2 SSM3J35MFV, Q3 SSM3K16FV, Q4 CSD15380F3T, U10 SN74LVC1T45DBVR, U11 DRV8838DSGR, U12 SN74LVC1T45DBVR, U13 TL3305AF260QG, U14 CDSOT23-SM712, U15 TPS63900DSKR, U16 TPS61299YBHR, U2 TPS22914BYFPR, U3 TPS22914BYFPR, U4 SN65HVD3082EDR, U5 TL3305AF260QG, U6 S-8240ADZ-M6T1U, U7 BME688, U8 TPS22914BYFPR

Commit message: commit before redesign
Connections:
- U15 pad 1: +3V3 -> +BATT
- U15 pad 2: +3V3 -> +BATT
Routing:
- net +3V3: track 171.5 -> 165.1 mm, vias 10 -> 9
- net +BATT: track 57.0 -> 61.9 mm
- net GND: vias 101 -> 102

Commit message: mutli soil sensor update
Other:
- board text added: "4 CORNER LID SCREWS: REFERENCE ONLY; DRILLS TBD"
- board text added: "6 INNER PCB BOSS CENTERS: 41.5 / 79.5 x 42.8 C-C"
- board text added: "ALL CIRCLE DIAMETERS ILLUSTRATIVE - VERIFY HARDWARE"
- board text added: "BFAB REFERENCE ONLY - CURRENT EDGES AND DRILLS UNCHANGED"
- board text added: "ENCLOSURE-FIT DRAFT: 90 x 58 mm, R5"
