File: Power.kicad_sch (KiCad schematic)
At the start: 33 parts, among them J3 Conn_01x01_Socket, J9 Conn_01x01_Socket, Q1 CSD15380F3T, Q2 SSM3J35MFV, Q3 SSM3K16FV, Q4 CSD15380F3T, U15 TPS63900DSKR, U16 TPS61299YBHR, U6 S-8240ADZ-M6T1U

Commit message: commit before redesign
Connections:
- net +3V3: no longer U15.1 (EN), U15.2 (SEL)
- net +BATT: now also U15.1 (EN), U15.2 (SEL)
Changed lines of the file:
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@@
 	)
 	(junction
+		(at 163.83 121.92)
+		(diameter 0)
+		(color 0 0 0 0)
+	)
+	(junction
 		(at 220.98 121.92)
 		(diameter 0)
@@
 	(wire
 		(pts
-			(xy 147.32 121.92) (xy 176.53 121.92)
+			(xy 147.32 121.92) (xy 163.83 121.92)
 		)
 		(stroke
@@
 	(wire
 		(pts
+			(xy 163.83 121.92) (xy 176.53 121.92)
+		)
+		(stroke
+			(width 0)
+			(type default)
+		)
+	)
+	(wire
+		(pts
 			(xy 147.32 113.03) (xy 147.32 121.92)
 		)
@@
 	(wire
 		(pts
-			(xy 163.83 129.54) (xy 163.83 132.08)
+			(xy 163.83 121.92) (xy 163.83 132.08)
 		)
 		(stroke
@@
 					(unit 1)
 				)
-			)
-		)
-	)
-	(symbol
-		(lib_id "power:+3V3")
-		(at 163.83 129.54 0)
-		(unit 1)
-		(body_style 1)
-		(exclude_from_sim no)
-		(in_bom yes)
-		(on_board yes)
-		(in_pos_files yes)
-		(dnp no)
-		(fields_autoplaced yes)
-		(property "Reference" "#PWR065"
-			(at 163.83 133.35 0)
-			(hide yes)
-			(show_name no)
-			(do_not_autoplace no)
-			(effects
-				(font
-					(size 1.27 1.27)
-				)
-			)
-		)
-		(property "Value" "+3V3"
-			(at 163.83 124.46 0)
-			(show_name no)
-			(do_not_autoplace no)
-			(effects
-				(font
-					(size 1.27 1.27)
-				)
-			)
-		)
-		(property "Footprint" ""
-			(at 163.83 129.54 0)
-			(hide yes)
-			(show_name no)
-			(do_not_autoplace no)
-			(effects
-				(font
-					(size 1.27 1.27)
-				)
-			)
-		)
-		(property "Datasheet" ""
-			(at 163.83 129.54 0)
-			(hide yes)
-			(show_name no)
-			(do_not_autoplace no)
-			(effects
-				(font
-					(size 1.27 1.27)
-				)
-			)
-		)
-		(property "Description" "Power symbol creates a global label with name \"+3V3\""
-			(at 163.83 129.54 0)
-			(hide yes)
-			(show_name no)
-			(do_not_autoplace no)
-			(effects
-				(font
-					(size 1.27 1.27)
-				)
-			)
-		)
-		(pin "1"
-		)
-		(instances
-			(project "SproutSync_SensorNode"
-				(path "/6b347550-6a02-4d2d-97d7-e1cbb1403859/8aac59c9-744f-46ff-a9bf-5095a50423d5"
-					(reference "#PWR065")
-					(unit 1)
-				)
