File: SproutSync_SensorNode.kicad_sch (KiCad schematic)
At the start: 0 parts

Commit message: mutli soil sensor update
Other:
- removed sheet Irrigation
- sheet AmbientSensors ports: added I2C_LVLSHFT_EN, LIGHT_GPIO, LIGHT_INT; removed none
Changed lines of the file:
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@@
-	)
-	(bus_entry
-		(at 130.81 127)
-		(size 2.54 -2.54)
-		(stroke
-			(width 0)
-			(type default)
-		)
 	)
 	(bus_entry
@@
 	)
 	(bus_entry
-		(at 130.81 116.84)
-		(size 2.54 -2.54)
-		(stroke
-			(width 0)
-			(type default)
-		)
-	)
-	(bus_entry
-		(at 130.81 123.19)
-		(size 2.54 -2.54)
-		(stroke
-			(width 0)
-			(type default)
-		)
-	)
-	(bus_entry
 		(at 128.27 81.28)
 		(size 2.54 -2.54)
@@
 	)
 	(bus_entry
+		(at 130.81 91.44)
+		(size 2.54 -2.54)
+		(stroke
+			(width 0)
+			(type default)
+		)
+	)
+	(bus_entry
+		(at 130.81 93.98)
+		(size 2.54 -2.54)
+		(stroke
+			(width 0)
+			(type default)
+		)
+	)
+	(bus_entry
 		(at 130.81 85.09)
 		(size 2.54 -2.54)
@@
 	)
 	(bus_entry
+		(at 130.81 87.63)
+		(size 2.54 -2.54)
+		(stroke
+			(width 0)
+			(type default)
+		)
+	)
+	(bus_entry
 		(at 130.81 44.45)
 		(size 2.54 2.54)
@@
 		)
 	)
-	(bus_entry
-		(at 130.81 114.3)
-		(size 2.54 -2.54)
-		(stroke
-			(width 0)
-			(type default)
-		)
-	)
-	(bus
-		(pts
-			(xy 130.81 113.03) (xy 130.81 114.3)
-		)
-		(stroke
-			(width 0)
-			(type default)
-		)
-	)
 	(wire
 		(pts
@@
 		)
 	)
-	(wire
-		(pts
-			(xy 133.35 114.3) (xy 151.13 114.3)
-		)
-		(stroke
-			(width 0)
-			(type default)
-		)
-	)
 	(bus
 		(pts
@@
 	(bus
 		(pts
-			(xy 130.81 119.38) (xy 130.81 123.19)
+			(xy 130.81 119.38) (xy 130.81 124.46)
 		)
 		(stroke
@@
 	(wire
 		(pts
+			(xy 133.35 86.36) (xy 133.35 85.09)
+		)
+		(stroke
+			(width 0)
+			(type default)
+		)
+	)
+	(wire
+		(pts
 			(xy 133.35 49.53) (xy 144.78 49.53)
 		)
@@
 	(bus
 		(pts
-			(xy 130.81 123.19) (xy 130.81 124.46)
-		)
-		(stroke
-			(width 0)
-			(type default)
-		)
-	)
-	(bus
-		(pts
-			(xy 130.81 114.3) (xy 130.81 116.84)
+			(xy 130.81 113.03) (xy 130.81 119.38)
 		)
 		(stroke
@@
 	(wire
 		(pts
+			(xy 133.35 88.9) (xy 151.13 88.9)
+		)
+		(stroke
+			(width 0)
+			(type default)
+		)
+	)
+	(wire
+		(pts
 			(xy 124.46 43.18) (xy 124.46 57.15)
 		)
@@
 		)
 	)
+	(wire
+		(pts
+			(xy 133.35 91.44) (xy 151.13 91.44)
+		)
+		(stroke
+			(width 0)
+			(type default)
+		)
+	)
 	(bus
 		(pts
@@
 	(wire
 		(pts
-			(xy 133.35 120.65) (xy 151.13 120.65)
-		)
-		(stroke
-			(width 0)
-			(type default)
-		)
-	)
-	(wire
-		(pts
-			(xy 133.35 111.76) (xy 151.13 111.76)
-		)
-		(stroke
-			(width 0)
-			(type default)
-		)
-	)
-	(wire
-		(pts
 			(xy 144.78 34.29) (xy 144.78 49.53)
 		)
@@
 	(wire
 		(pts
-			(xy 133.35 124.46) (xy 151.13 124.46)
-		)
-		(stroke
-			(width 0)
-			(type default)
-		)
-	)
-	(wire
-		(pts
 			(xy 124.46 57.15) (xy 151.13 57.15)
 		)
@@
 		)
 	)
+	(wire
+		(pts
+			(xy 133.35 86.36) (xy 151.13 86.36)
+		)
+		(stroke
+			(width 0)
+			(type default)
+		)
+	)
 	(bus
 		(pts
@@
 		(pts
 			(xy 130.81 44.45) (xy 130.81 46.99)
-		)
-		(stroke
-			(width 0)
-			(type default)
-		)
-	)
-	(bus
-		(pts
-			(xy 130.81 116.84) (xy 130.81 119.38)
 		)
 		(stroke
@@
 		)
 	)
-	(label "PAD6"
-		(at 134.62 124.46 0)
-		(effects
-			(font
-				(size 1.27 1.27)
-			)
-			(justify left bottom)
-		)
-	)
 	(label "PAD49"
 		(at 134.62 78.74 0)
@@
 		)
 	)
-	(label "PAD2"
-		(at 134.62 111.76 0)
-		(effects
-			(font
-				(size 1.27 1.27)
-			)
-			(justify left bottom)
-		)
-	)
 	(label "PAD48"
 		(at 134.62 82.55 0)
-		(effects
-			(font
-				(size 1.27 1.27)
-			)
-			(justify left bottom)
-		)
-	)
-	(label "PAD4"
-		(at 134.62 114.3 0)
-		(effects
-			(font
-				(size 1.27 1.27)
-			)
-			(justify left bottom)
-		)
-	)
-	(label "PAD5"
-		(at 134.62 120.65 0)
 		(effects
 			(font
@@
 			)
 		)
+		(pin "I2C_LVLSHFT_EN" output
+			(at 151.13 86.36 180)
+			(effects
+				(font
+					(size 1.27 1.27)
+				)
+				(justify left)
+			)
+		)
+		(pin "LIGHT_GPIO" output
+			(at 151.13 88.9 180)
+			(effects
+				(font
+					(size 1.27 1.27)
+				)
+				(justify left)
+			)
+		)
+		(pin "LIGHT_INT" output
+			(at 151.13 91.44 180)
+			(effects
+				(font
+					(size 1.27 1.27)
+				)
+				(justify left)
+			)
+		)
 		(instances
 			(project "SproutSync_SensorNode"
 				(path "/6b347550-6a02-4d2d-97d7-e1cbb1403859"
-					(page "4")
+					(page "3")
 				)
 			)
@@
 			(project "SproutSync_SensorNode"
 				(path "/6b347550-6a02-4d2d-97d7-e1cbb1403859"
-					(page "6")
+					(page "4")
 				)
 			)
@@
 	)
 	(sheet
-		(at 151.13 108.585)
-		(size 25.4 25.4)
-		(exclude_from_sim no)
-		(in_bom yes)
-		(on_board yes)
-		(dnp no)
-		(fields_autoplaced yes)
-		(stroke
-			(width 0.1524)
-			(type solid)
-		)
-		(fill
-			(color 0 0 0 0)
-		)
-		(property "Sheetname" "Irrigation"
-			(at 151.13 107.8734 0)
-			(show_name no)
-			(do_not_autoplace no)
-			(effects
-				(font
-					(size 1.27 1.27)
-				)
-				(justify left bottom)
-			)
-		)
-		(property "Sheetfile" "Irrigation.kicad_sch"
-			(at 151.13 134.5696 0)
-			(show_name no)
-			(do_not_autoplace no)
-			(effects
-				(font
-					(size 1.27 1.27)
-				)
-				(justify left top)
-			)
-		)
-		(pin "FLOW_PPS" output
-			(at 151.13 120.65 180)
-			(effects
-				(font
-					(size 1.27 1.27)
-				)
-				(justify left)
-			)
-		)
-		(pin "FLOW_SNS_ENA" input
-			(at 151.13 124.46 180)
-			(effects
-				(font
-					(size 1.27 1.27)
-				)
-				(justify left)
-			)
-		)
-		(pin "IRRI_ENA" input
-			(at 151.13 114.3 180)
-			(effects
-				(font
-					(size 1.27 1.27)
-				)
-				(justify left)
-			)
-		)
-		(pin "IRRI_PHS" input
-			(at 151.13 111.76 180)
-			(effects
-				(font
-					(size 1.27 1.27)
-				)
-				(justify left)
-			)
-		)
-		(instances
-			(project "SproutSync_SensorNode"
-				(path "/6b347550-6a02-4d2d-97d7-e1cbb1403859"
-					(page "7")
-				)
-			)
-		)
-	)
-	(sheet
 		(at 151.13 24.765)
 		(size 25.4 20.32)
@@
 			(project "SproutSync_SensorNode"
 				(path "/6b347550-6a02-4d2d-97d7-e1cbb1403859"
-					(page "8")
+					(page "6")
 				)
 			)
@@
 			(project "SproutSync_SensorNode"
 				(path "/6b347550-6a02-4d2d-97d7-e1cbb1403859"
-					(page "3")
-				)
-			)
+					(page "7")
+				)
+			)
